Commit message: sdfsdf

File: description/robot_core.xacro (robot description, xacro)
@@ -21,9 +21,9 @@
         <parent link="base_link"/>
         <child link="chassis"/>
-        <origin xyz="-0.1 0 0"/>
+        <origin xyz="0.1 0 0"/>
     </joint>
     <link name="chassis">
         <visual>
-            <origin xyz="0.25 0 0.075"/>
+            <origin xyz="-0.25 0 0.075"/>
             <geometry>
                 <box size="0.5 0.3 0.15"/>
@@ -32,5 +32,5 @@
         </visual>
         <collision>
-            <origin xyz="0.25 0 0.075"/>
+            <origin xyz="-0.25 0 0.075"/>
             <geometry>
                 <box size="0.5 0.3 0.15"/>
@@ -38,7 +38,10 @@
         </collision>
         <xacro:inertial_box mass="0.5" x="0.5" y="0.3" z="0.15">
-            <origin xyz="0.25 0 0.075" rpy="0 0 0"/>
+            <origin xyz="-0.25 0 0.075" rpy="0 0 0"/>
         </xacro:inertial_box>
     </link>
+    <gazebo reference="chassis">
+        <material>Gazebo/White</material>
+    </gazebo>
     <!-- LEFT WHEEL LINK -->
     <joint name="left_wheel_joint" type="continuous">
@@ -64,4 +67,7 @@
         </xacro:inertial_cylinder>
     </link>
+    <gazebo reference="left_wheel">
+        <material>Gazebo/Blue</material>
+    </gazebo>
     <!-- RIGHT WHEEL LINK -->
     <joint name="right_wheel_joint" type="continuous">
@@ -87,9 +93,12 @@
         </xacro:inertial_cylinder>
     </link>
+    <gazebo reference="right_wheel">
+        <material>Gazebo/Blue</material>
+    </gazebo>
     <!-- CASTER WHEEL LINK -->
     <joint name="caster_wheel_joint" type="fixed">
         <parent link="chassis"/>
         <child link="caster_wheel"/>
-        <origin xyz="0.4 0 0"/>
+        <origin xyz="-0.4 0 0"/>
     </joint>
     <link name="caster_wheel">
@@ -109,3 +118,8 @@
         </xacro:inertial_sphere>
     </link>
+    <gazebo reference="caster_wheel">
+        <material>Gazebo/Black</material>
+        <mu1 value="0.001"/>
+        <mu2 value="0.001"/>
+    </gazebo>
 </robot>
