Commit message: stuff

File: description/lidar.xacro (robot description, xacro)
@@ -2,5 +2,5 @@
 <robot xmlns:xacro="http://www.ros.org/wiki/xacro"  name="robot">
     <joint name="laser_joint" type="fixed">
-        <origin xyz="-0.05 0 0.175" rpy="0 0 0"/>
+        <origin xyz="-0.35 0 0.175" rpy="0 0 0"/>
         <parent link="chassis"/>
         <child link="laser_frame"/>

File: description/robot_core.xacro (robot description, xacro)
@@ -30,5 +30,5 @@
             <origin xyz="-0.25 0 0.075"/>
             <geometry>
-                <box size="0.5 0.3 0.15"/>
+                <box size="0.3 0.3 0.15"/>
             </geometry>
             <material name="white"/>
